File: FC_hardware/FC/FC.kicad_sch (KiCad schematic)
At the start: 78 parts, among them J1 Pin_01x04, J10 GND, J11 GND, J12 GND, J13 Pin_02x03, J14 Pin_01x03, J15 Pin_01x03, J16 PB2, J17 PC9, J18 PC8, J19 PB7, J2 USB4105GFA120, J20 PB6, J21 PA8, J22 PC11, J23 PC10, J24 PC12, J25 PB10, J26 PC7, J27 PC6, J3 530480810, J4 BAT, J5 5V, J6 5V, J7 3V3, J8 3V3, J9 GND, Q1 BC807W, U1 MP2348, U2 AMS1117-3.3, U3 STM32F446RETx, U4 MPU-9250, U5 DPS368XTSA1, U6 Ai-Thinker-Ra-02, Y1 ABM8G-25MHZ

Commit message: 0201 changed to 0603
Parts:
- C10, C3, C9: footprint Capacitor_SMD:C_0201_0603Metric -> Capacitor_SMD:C_0603_1608Metric
- R1, R10, R11, R12, R13, R14, R15, R16, R17, R18, R2, R3, R4, R5, R6, R7, R8, R9: footprint Resistor_SMD:R_0201_0603Metric -> Resistor_SMD:R_0603_1608Metric

Commit message: Pin config changed, LoRa module removed from board
Parts:
- removed J13: Pin_02x03, Connector_PinHeader_1.27mm:PinHeader_2x03_P1.27mm_Vertical, symbol Connector_Generic:Conn_01x06
- removed J14: Pin_01x03, Connector_PinHeader_1.27mm:PinHeader_1x03_P1.27mm_Vertical, symbol Connector_Generic:Conn_01x03
- removed U6: Ai-Thinker-Ra-02, RF_Module:Ai-Thinker-Ra-01-LoRa, symbol RF_Module:Ai-Thinker-Ra-02
- added C18, C19, C20, C21, C22: 0.1uF, Capacitor_SMD:C_0603_1608Metric, symbol Device:C
- added J13: 530481410, footprints:MOLEX_530481410, symbol 530481410:530481410
Connections:
- net LORA_NSS is gone; now on net LORA_RST: U3.20 (PA4)
- net 3V3: now also C15.2, U5.1 (GND), U5.7 (GND), C18.2, C19.2, C20.2, C21.2, C22.1, J13.2 (3V3); no longer C14.1, C15.1, U5.6 (VDDIO), U5.8 (VDD)
- net 5V: now also C14.1, J13.3 (5V)
- net ADC_I: now also U3.8 (PC0); no longer U3.10 (PC2)
- net GEN_SCK: now also U3.55 (PB3); no longer U3.51 (PC10)
- net GND: now also C15.1, R17.1, U5.6 (VDDIO), U5.8 (VDD), C18.1, C19.1, C20.1, C21.1, C22.2, J13.1 (GND); no longer C15.2, R18.1, U4.22 (~{CS}), U5.1 (GND), U5.7 (GND)
- net GPS_RX: now also J13.6 (GPS_RX)
- net GPS_TX: now also J13.5 (GPS_TX)
- net LORA_IRQN: now also J13.13 (LORA_IRQ)
- net LORA_RST: now also J13.12 (LORA_RST); no longer U3.21 (PA5)
- net MAG_SCL: now also J13.8 (MAG_SCL)
- net MAG_SDA: now also J13.7 (MAG_SDA)
- net SBUS_RX: now also R17.2; no longer R18.2
- net ESC_RX_MCU: now reaches JP2.2 (B), U3.25 (PC5)
- net at Q1.1 (B): now also R18.1; no longer R17.1
- net BAT_VIN: now reaches C1.1, F1.2, R5.1, U1.2 (VIN)
- net SW: now reaches C6.2, L1.1, U1.3 (SW)
- net OSC_IN: now reaches C9.2, U3.5 (PH0), Y1.1
- net OSC_OUT: now reaches C10.1, U3.6 (PH1), Y1.3
- net VCAP_1: now reaches C8.2, U3.30 (VCAP_1)
- net LED: now reaches D3.2 (A), U3.33 (PB12)
- net IMU_CS: now reaches U3.50 (PA15)
- net IMU_CS: now also U4.22 (~{CS})
- net BOOT: now reaches JP1.2 (B), R7.1, U3.60 (BOOT0)
- net NRST: now reaches R6.1, S1.1_1, S1.1_2, U3.7 (NRST)
- net IMU_MISO renamed IMU_BAR_MISO
- net IMU_BAR_MISO: now also U5.5 (SDO)
- net IMU_MOSI renamed IMU_BAR_MOSI
- net IMU_BAR_MOSI: now also U5.3 (SDI)
- net IMU_SCK renamed IMU_BAR_SCK
- net IMU_BAR_SCK: now also U3.21 (PA5), U5.4 (SCK); no longer U3.55 (PB3)
- net LORA_BAR_MISO renamed LORA_MISO
- net LORA_MISO: now also J13.10 (LORA_MISO); no longer U5.5 (SDO)
- net LORA_BAR_MOSI renamed LORA_MOSI
- net LORA_MOSI: now also J13.9 (LORA_MOSI); no longer U5.3 (SDI)
- net LORA_BAR_SCK renamed LORA_SCK
- net LORA_SCK: now also J13.11 (LORA_SCK); no longer U5.4 (SCK)
- new net: J13.4 (SBUS_RX), R18.2
- no-connect marks 16 -> 12
Other:
- note added: "IMU/Barometer"
- note added: "LoRa/GPS/SBUS"
- note removed: "GPS/SBUS"
- note removed: "IMU"
- note removed: "LoRa/Barometer"
- moved on the sheet: C12, C13, C14, J15, J16, J17, J18, J19, J20, J21, J22, J23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

Commit message: Improve schematic, settings
Parts:
- added H1, H2, H3, H4: MountingHole, MountingHole:MountingHole_2.2mm_M2, symbol Mechanical:MountingHole
- added U6: USBLC6-2SC6, Package_TO_SOT_SMD:SOT-23-6, symbol Power_Protection:USBLC6-2SC6
Connections:
- net GND: now also R9.2, S1.1_1, S1.1_2, U5.1 (GND), U5.7 (GND), U6.2 (GND); no longer R9.1, S1.2_1, S1.2_2, U5.6 (VDDIO), U5.8 (VDD)
- net NRST: now also S1.2_1, S1.2_2; no longer S1.1_1, S1.1_2
- net USB_DP: now also U6.1 (I/O1); no longer J2.A6 (DP1), J2.B6 (DP2)
- net VBUS: now reaches D1.2 (A), J2.A4_B9 (VBUS), J2.B4_A9 (VBUS)
- net VBUS: now also U6.5 (VBUS)
- net at J2.A5 (CC1): now also R9.1; no longer R9.2
- net 3V3 renamed +3V3
- net +3V3: now also U5.6 (VDDIO), U5.8 (VDD); no longer U5.1 (GND), U5.7 (GND)
- net 5V renamed +5V
- net BAT renamed +BATT
- net USB_DM renamed USB_DC_N
- net USB_DC_N: now also U6.4 (I/O2); no longer U3.44 (PA11)
- new net USB_DC_P: J2.A6 (DP1), J2.B6 (DP2), U6.6 (I/O1)
- new net USB_DN: U3.44 (PA11), U6.3 (I/O2)
Other:
- moved on the sheet: C10, C11, C14, C15, C16, C18, C19, C20, C21, C22, C5, C7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

Commit message: Update stm pin config, clean up schematic
Parts:
- removed J16: PB2, footprints:1.27mm_pin, symbol Connector:Conn_01x01_Pin
- removed J22: PC11, footprints:1.27mm_pin, symbol Connector:Conn_01x01_Pin
- removed J23: PC10, footprints:1.27mm_pin, symbol Connector:Conn_01x01_Pin
- removed JP2: ESC_TEL, Jumper:SolderJumper-2_P1.3mm_Open_RoundedPad1.0x1.5mm, symbol Jumper:Jumper_2_Small_Open
- added J9: PC9, footprints:1.27mm_pin, symbol Connector:Conn_01x01_Pin
- added NT1: NetTie_2, NetTie:NetTie-2_SMD_Pad0.5mm, symbol Device:NetTie_2
- H1, H2, H3, H4: footprint MountingHole:MountingHole_2.2mm_M2 -> MountingHole:MountingHole_3.2mm_M3
- renumbered C4 to C10, C9 to C11, C10 to C12, C14 to C13, C22 to C14, C8 to C15, C11 to C16, C18 to C17, C19 to C18, C20 to C19, C7 to C2, C21 to C20, C17 to C21, C16 to C22, C5 to C3, C12 to C4, C13 to C5, C15 to C7, C3 to C8, C2 to C9, D2 to D1, D3 to D2, D1 to D3, J13 to J1, J4 to J10, J5 to J11, J6 to J12, J24 to J13, J25 to J14, J26 to J15, J27 to J16, J15 to J17, J7 to J18, J8 to J19, J9 to J20, J10 to J21, J12 to J22, J11 to J23, J3 to J24, J1 to J3, J21 to J4, J20 to J5, J19 to J6, J18 to J7, J17 to J8, JP1 to JP2, R5 to R1, R6 to R10, R15 to R11, R7 to R12, R18 to R13, R8 to R14, R17 to R15, R12 to R16, R11 to R17, R10 to R18, R13 to R2, R4 to R3, R3 to R4, R1 to R5, R2 to R6, R9 to R7, R14 to R8, R16 to R9, U2 to U1, U4 to U2, U1 to U3, U5 to U4, U3 to U5
Connections:
- net GEN_MISO is gone; now on net GPS_RX: U5.52 (PC11)
- net GEN_SCK is gone; now on net LORA_SCK: U5.55 (PB3)
- net +3V3: now also J3.1 (Pin_1); no longer J3.4 (3V3)
- net BAT_VIN: now also NT1.1; no longer R1.1
- net GND: now also D2.1 (K), J3.4 (Pin_4); no longer J3.1 (GND), R8.1
- net GPS_RX: no longer U5.17 (PA3)
- net GPS_TX: now also U5.51 (PC10); no longer U5.16 (PA2)
- net IMU_BAR_MISO: now also U5.35 (PB14); no longer U5.56 (PB4)
- net IMU_BAR_MOSI: now also U5.36 (PB15); no longer U5.57 (PB5)
- net IMU_BAR_SCK: now also U5.34 (PB13); no longer U5.21 (PA5)
- net IMU_CS: now also U5.37 (PC6); no longer U5.50 (PA15)
- net IMU_IRQN: now also U5.33 (PB12); no longer U5.54 (PD2)
- net LORA_IRQN: now also U5.2 (PC13); no longer U5.24 (PC4)
- net LORA_MISO: now also U5.56 (PB4); no longer U5.35 (PB14)
- net LORA_MOSI: now also U5.57 (PB5); no longer U5.36 (PB15)
- net LORA_RST: now also U5.3 (PC14); no longer U5.20 (PA4)
- net LORA_SCK: no longer U5.34 (PB13)
- net MAG_SCL: now also U5.58 (PB6); no longer U5.61 (PB8)
- net MAG_SDA: now also U5.59 (PB7); no longer U5.62 (PB9)
- net SBUS_RX: now also U5.54 (PD2); no longer U5.15 (PA1)
- net STATUS_LED: now reaches U5.10 (PC2)
- net STATUS_LED: now also R8.1
- net VBAT_ADC: now reaches U5.14 (PA0)
- net VBAT_ADC: now also C21.1, R16.2, R17.2
- net at R8.2: now also D2.2 (A); no longer D2.1 (K)
- net ADC_I renamed IBAT_ADC
- net IBAT_ADC: now also U5.15 (PA1); no longer U5.8 (PC0)
- removed net ADC_U: C21.1, R16.2, R17.2, U5.9 (PC1)
- net BAR_CSB renamed BAR_CS
- net BAR_CS: now also U5.38 (PC7); no longer U5.2 (PC13)
- net DEBUG_RX renamed DEBUG_UART1_RX
- net DEBUG_TX renamed DEBUG_UART1_TX
- net ESC_RX: no longer names the net of J24.1
- net ESC_RX_MCU: no longer names the net of U5.25 (PC5)
- net GEN_MOSI renamed GEN_TIM2_CH4
- net GEN_TIM2_CH4: now also J7.1 (Pin_1)
- net GEN_RX renamed GEN_UART2_RX
- net GEN_UART2_RX: now also U5.17 (PA3); no longer U5.38 (PC7)
- net GEN_SCL renamed GEN_I2C3_SCL
- net GEN_I2C3_SCL: now also U5.41 (PA8); no longer U5.29 (PB10)
- net GEN_SDA renamed GEN_I2C3_SDA
- net GEN_I2C3_SDA: now also U5.40 (PC9); no longer U5.53 (PC12)
- net GEN_TX renamed GEN_UART2_TX
- net GEN_UART2_TX: now also U5.16 (PA2); no longer U5.37 (PC6)
- removed net LED: D2.2 (A), U5.33 (PB12)
- net OSC_IN renamed RCC_OSC_IN
- net OSC_OUT renamed RCC_OSC_OUT
- net SWCLK renamed SYS_JTCK-SWCLK
- net SYS_JTCK-SWCLK: now also J3.3 (Pin_3); no longer J3.2 (CLK)
- net SWDIO renamed SYS_JTMS-SWDIO
- net SYS_JTMS-SWDIO: now also J3.2 (Pin_2); no longer J3.3 (DIO)
- net TIM1_1 renamed GEN_TIM2_CH1
- net GEN_TIM2_CH1: now also U5.21 (PA5); no longer U5.41 (PA8)
- net TIM4_1 renamed GEN_TIM2_CH2
- net GEN_TIM2_CH2: now also U5.62 (PB9); no longer U5.58 (PB6)
- net TIM4_2 renamed GEN_TIM2_CH3
- net GEN_TIM2_CH3: now also U5.29 (PB10); no longer U5.59 (PB7)
- net TIM8_3 renamed GEN_TIM8_CH3
- net GEN_TIM8_CH3: now also J8.1 (Pin_1); no longer J7.1 (Pin_1)
- removed net TIM8_4: J8.1 (Pin_1), U5.40 (PC9)
- net USB_DN renamed USB_OTG_FS_DN
- net USB_DP renamed USB_OTG_FS_DP
- new net: NT1.2, R1.1
- new net GEN_TIM10_CH1: J9.1 (Pin_1), U5.61 (PB8)
- new net UART5_TX_NC: U5.53 (PC12)
- no-connect marks 12 -> 16
Other:
- note added: "Debug"
- note added: "Generic I2C, UART"
- note added: "Generic Timers / GPIO"
- note added: "MCU Oscillator"
- moved on the sheet: C1, C10, C11, C12, C14, C15, C16, C17, C18, C19, C2, C20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

Commit message: Dump pcb design
Parts:
- removed J1: 530481410, footprints:MOLEX_530481410, symbol 530481410:530481410
- removed J17: Pin_01x03, Connector_PinHeader_1.27mm:PinHeader_1x03_P1.27mm_Vertical, symbol Connector_Generic:Conn_01x03
- removed J24: 530480810, footprints:MOLEX_530480810, symbol 530480810:530480810
- removed J3: Pin_01x04, Connector_PinHeader_1.27mm:PinHeader_1x04_P1.27mm_Vertical, symbol Connector_Generic:Conn_01x04
- removed NT1: NetTie_2, NetTie:NetTie-2_SMD_Pad0.5mm, symbol Device:NetTie_2
- added C23: 10nF, Capacitor_SMD:C_0603_1608Metric, symbol Device:C
- added C24, C25: 10uF, Capacitor_SMD:C_0603_1608Metric, symbol Device:C
- added FB1: 120R, Inductor_SMD:L_1206_3216Metric, symbol Device:FerriteBead
- added J1: Conn_01x14, Connector_JST:JST_SH_SM14B-SRSS-TB_1x14-1MP_P1.00mm_Horizontal, symbol Connector_Generic:Conn_01x14
- added J24: SM08B-SRSS-TB, JST_SH_SM08B-SRSS-TB_1x08-1MP_P1.00mm_Horizontal, symbol SM08B-SRSS-TB:SM08B-SRSS-TB
- added J25: Conn_01x06, Connector_PinHeader_1.27mm:PinHeader_1x06_P1.27mm_Vertical, symbol Connector_Generic:Conn_01x06
- J10: footprint footprints:1.27mm_pin -> Connector_PinHeader_2.00mm:PinHeader_1x01_P2.00mm_Vertical
Connections:
- net +3V3: now also R11.1, C25.2, FB1.2, J1.13 (Pin_13), J25.6 (Pin_6); no longer R11.2, U5.13 (VDDA)
- net +5V: now also J1.12 (Pin_12)
- net +BATT: now also J24.2
- net BAT_VIN: now also R1.1
- net DEBUG_UART1_RX: now also J25.3 (Pin_3)
- net DEBUG_UART1_TX: now also J25.2 (Pin_2)
- net ESC_1: now also J24.3
- net ESC_2: now also J24.4
- net ESC_3: now also J24.5
- net ESC_4: now also J24.6
- net GND: now also C23.1, C24.1, C25.1, J1.14 (Pin_14), J24.1, J25.1 (Pin_1)
- net GPS_RX: now also J1.3 (Pin_3)
- net GPS_TX: now also J1.2 (Pin_2)
- net LORA_IRQN: now also J1.10 (Pin_10)
- net LORA_MISO: now also J1.6 (Pin_6)
- net LORA_MOSI: now also J1.7 (Pin_7)
- net LORA_RST: now also J1.11 (Pin_11)
- net LORA_SCK: now also J1.5 (Pin_5)
- net MAG_SCL: now also J1.8 (Pin_8)
- net MAG_SDA: now also R11.2, J1.9 (Pin_9); no longer R11.1
- net SYS_JTCK-SWCLK: now also J25.5 (Pin_5)
- net SYS_JTMS-SWDIO: now also J25.4 (Pin_4)
- net at R13.2: now also J1.4 (Pin_4)
- net at R18.2: now also J24.7
- new net VDDA: C23.2, C24.2, FB1.1, U5.13 (VDDA)
Other:
- moved on the sheet: C13, C14, Q1, R10, R11, R13, R15, R9, S1

Commit message: Finalize design
Parts:
- removed J13: PC12, footprints:1.27mm_pin, symbol Connector:Conn_01x01_Pin
- removed J14: PB10, footprints:1.27mm_pin, symbol Connector:Conn_01x01_Pin
- removed J15: PC7, footprints:1.27mm_pin, symbol Connector:Conn_01x01_Pin
- removed J16: PC6, footprints:1.27mm_pin, symbol Connector:Conn_01x01_Pin
- removed J4: PA8, footprints:1.27mm_pin, symbol Connector:Conn_01x01_Pin
- removed J8: PC9, footprints:1.27mm_pin, symbol Connector:Conn_01x01_Pin
- added J3, J4: Conn_02x02_Counter_Clockwise, Connector_PinHeader_1.27mm:PinHeader_2x02_P1.27mm_Vertical, symbol Connector_Generic:Conn_02x02_Counter_Clockwise
- J25: footprint Connector_PinHeader_1.27mm:PinHeader_1x06_P1.27mm_Vertical -> Connector_PinHeader_1.27mm:PinHeader_2x03_P1.27mm_Vertical
Connections:
- net +3V3: now also J25.3 (Pin_3); no longer J25.6 (Pin_6)
- net DEBUG_UART1_RX: now also J25.6 (Pin_6); no longer J25.3 (Pin_3)
- net DEBUG_UART1_TX: now also J25.5 (Pin_5); no longer J25.2 (Pin_2)
- net GEN_I2C3_SCL: now also J3.2 (Pin_2)
- net GEN_I2C3_SDA: now also J3.1 (Pin_1)
- net GEN_TIM2_CH1: now also J4.3 (Pin_3)
- net GEN_TIM8_CH3: now also J3.3 (Pin_3)
- net GEN_UART2_RX: now also J4.1 (Pin_1)
- net GEN_UART2_TX: now also J4.2 (Pin_2)
- net GND: now also J3.4 (Pin_4), J4.4 (Pin_4)
- net SYS_JTCK-SWCLK: now also J25.2 (Pin_2); no longer J25.5 (Pin_5)
- no-connect marks 16 -> 15
Other:
- moved on the sheet: J25, J9

Commit message: farnell BOM
Parts:
- D3: Farnell (none) -> https://hu.farnell.com/diodes-inc/b320a-13-f/diode-rec-scho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
- F1: Farnell (none) -> https://hu.farnell.com/vishay/mfu0805ff04000p100/fuse-0805-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
- FB1, J10, J11, J12, J18, J19, J20, J21, J22, J23, J5, J6, J7, J9, JP2, U2: now left out of the parts list
- J1: Farnell (none) -> https://hu.farnell.com/jst-japan-solderless-terminals/sm14b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
- J2: Farnell (none) -> https://hu.farnell.com/gct-global-connector-technology/usb4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
- J24: Farnell (none) -> https://hu.farnell.com/jst-japan-solderless-terminals/sm08b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
- J25: Farnell (none) -> https://hu.farnell.com/samtec/tms-106-02-g-s-ra/header-1-27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
- J3, J4: Farnell (none) -> https://hu.farnell.com/samtec/ftsh-106-02-f-d-ra/conn-r-a-h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
- L1: Farnell (none) -> https://hu.farnell.com/yageo/bwvs005050404r7m00/inductor-4-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
- Q1: Farnell (none) -> https://hu.farnell.com/nexperia/bc807-25w-115/transistor-bi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
- S1: Farnell (none) -> https://hu.farnell.com/panasonic/evqp7l01p/tactile-sw-spst-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
- U3: Farnell (none) -> https://hu.farnell.com/monolithic-power-systems-mps/mp2348g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
- U4: Farnell (none) -> https://hu.farnell.com/infineon/dps368xtsa1/pressure-sensor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
- U5: Farnell (none) -> https://hu.farnell.com/stmicroelectronics/stm32f446ret6/mcu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
- U6: Farnell (none) -> https://hu.farnell.com/stmicroelectronics/usblc6-2sc6/esd-p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
- Y1: Farnell (none) -> https://hu.farnell.com/abracon/abm8g-25-000mhz-18-d2y-t/cry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
